File: latte/latte.kicad_sch (KiCad schematic)
At the start: 85 parts, among them J1 SOIC bite, J2 USB_C_Receptacle_USB2.0, J3 USB_C_Receptacle_USB2.0, J4 USB_C_2.0, J5 USB_A, J6 OUT1, J7 OUT2, J8 SENSE1, J9 SENSE2, Q1 IRLML0030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

Commit message: Rough layout done
Parts:
- removed D11: LED, symbol Device:LED
- removed D12: BAV99, Package_TO_SOT_SMD:SOT-23, symbol Diode:BAV99
- removed D15, D3, D4: PMEG3020EH, Diode_SMD:D_SOD-123F, symbol Diode:PMEG3020EH
- removed F2: 1A, symbol Device:Polyfuse
- removed J7: OUT2, symbol Connector_Generic:Conn_01x02
- removed J9: SENSE2, symbol Connector_Generic:Conn_01x02
- removed Q2: IRLML0030, Package_TO_SOT_SMD:SOT-23, symbol Transistor_FET:IRLML0030
- removed R12, R13, R14: 1M, symbol Device:R
- removed R21, R26: 10k, symbol Device:R
- removed R23: 100R, symbol Device:R
- removed R25: 4k7, symbol Device:R
- removed R28: DNP, symbol Device:R
- removed U4, U5, U7, U8: USBLC6-2P6, Package_TO_SOT_SMD:SOT-666, symbol Power_Protection:USBLC6-2P6
- removed U6: FSUSB30MUX, Package_SO:MSOP-10_3x3mm_P0.5mm, symbol Interface_USB:FSUSB30MUX
- added C19: 100n, Capacitor_SMD:C_0603_1608Metric, symbol Device:C
- added D3: BAV99, Package_TO_SOT_SMD:SOT-23, symbol Diode:BAV99
- added H1, H2, H3, H4: MountingHole_Pad, MountingHole:MountingHole_3.2mm_M3_Pad_Via, symbol Mechanical:MountingHole_Pad
- added R30: 22k, Resistor_SMD:R_0603_1608Metric, symbol Device:R
- added R31: 33k, Resistor_SMD:R_0603_1608Metric, symbol Device:R
- added U4, U5, U7, U8: USBLC6-2SC6, Package_TO_SOT_SMD:SOT-23-6, symbol Power_Protection:USBLC6-2SC6
- added U6: FSUSB30UMX, Package_DFN_QFN:UQFN-10_1.3x1.8mm_P0.4mm, symbol onsemi:FSUSB30UMX
- C1, C10, C11, C12, C13, C14, C15, C16, C17, C18, C2, C3, C4, C7, C8, C9: footprint (none) -> Capacitor_SMD:C_0603_1608Metric
- C5, C6: footprint Capacitor_SMD:C_0402_1005Metric -> Capacitor_SMD:C_0603_1608Metric
- D10, D5, D6, D7, D8, D9: footprint (none) -> LED_SMD:LED_0603_1608Metric
- F1: footprint (none) -> Fuse:Fuse_0603_1608Metric
- J1: footprint (none) -> soicbite:SOIC_clipProgSmall
- J2, J3, J4: footprint (none) -> Connector_USB:USB_C_Receptacle_XKB_U262-16XN-4BVC11
- J5: footprint (none) -> Connector_USB:USB_A_Molex_67643_Horizontal
- J6, J8: footprint (none) -> TerminalBlock:TerminalBlock_bornier-2_P5.08mm
- R1, R10, R11, R15, R16, R17, R18, R19, R2, R20, R22, R24, R27, R29, R3, R4, R5, R6, R7, R8, R9: footprint (none) -> Resistor_SMD:R_0603_1608Metric
- SW1: footprint (none) -> Button_Switch_SMD:SW_SPST_EVQPE1
Connections:
- net +3V3: now also C18.1, D3.2 (A), U6.9 (VCC)
- net +5V: no longer C18.1
- net DUT_USB_D+: now also U5.6 (I/O1), U6.3 (D+)
- net DUT_USB_D-: now also U5.4 (I/O2), U6.5 (D-)
- net DUT_USB_S: now also U6.10 (S)
- net GND: now also C19.2, D3.1 (K), R31.2, U4.2 (GND), U5.2 (GND), U6.4 (GND), U7.2 (GND), U8.5 (VBUS)
- net USB_D+: now also U4.4 (I/O2)
- net USB_D-: now also U4.6 (I/O1)
- net ~{DUT_USB_OE}: now also U6.8 (~{OE})
- net at J2.A7 (D-), J2.B7 (D-): now also U5.1 (I/O1)
- net at J2.A6 (D+), J2.B6 (D+): now also U5.3 (I/O2)
- net VBUS: now reaches J2.A4 (VBUS), J2.A9 (VBUS), J2.B4 (VBUS), J2.B9 (VBUS), R1.2, R2.1
- net VBUS: now also D2.2 (A), J4.A4 (VBUS), J4.A9 (VBUS), J4.B4 (VBUS), J4.B9 (VBUS), J5.1 (VBUS), R10.2, R11.1, R30.1, U5.5 (VBUS), U7.5 (VBUS), U8.2 (GND); no longer D1.2 (A)
- net at J3.A7 (D-), J3.B7 (D-): now also U4.1 (I/O1)
- net at J3.A6 (D+), J3.B6 (D+): now also U4.3 (I/O2)
- net at J3.A4 (VBUS), J3.A9 (VBUS), J3.B4 (VBUS)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: now also D1.2 (A), U4.5 (VBUS); no longer D2.2 (A)
- net VBUS_SENSE: now reaches U1.40 (GPIO28_ADC2)
- net VBUS_SENSE: now also C19.1, D3.3 (K), R30.2, R31.1
- net at J5.3 (D+): now also U8.6 (I/O1)
- net at J5.2 (D-): now also U8.4 (I/O2)
- net at J4.A6 (D+), J4.B6 (D+): now also U7.3 (I/O2)
- net at J4.A7 (D-), J4.B7 (D-): now also U7.1 (I/O1)
- net TOUCH1: no longer names the net of U1.29 (GPIO18)
- net TOUCH2: no longer names the net of U1.32 (GPIO21)
- net TOUCH3: no longer names the net of U1.36 (GPIO24)
- new net: U6.1 (HSD1+), U8.1 (I/O1)
- new net: U6.2 (HSD2+), U7.4 (I/O2)
- new net: U6.6 (HSD2-), U7.6 (I/O1)
- new net: U6.7 (HSD1-), U8.3 (I/O2)
- no-connect marks 22 -> 31
Other:
- moved on the sheet: D13, J8, R27, R29
